File: cat_toilet.sch (KiCad schematic (older format))
At the start: 28 parts, among them J1 Conn_01x02, J2 ISP, SW1 EN Btn, SW2 EN Btn, U1 NCP187, U2 USB_CType_6Pin, U3 MCP73831, U4 ESP32-WROOM-32E

Commit message: 2021-08-12 2
Parts:
- added D3: LED, LED_SMD:LED_0805_2012Metric_Pad1.15x1.40mm_HandSolder, symbol Device:LED
- added R7: 1k, Resistor_SMD:R_0603_1608Metric_Pad0.98x0.95mm_HandSolder, symbol cat_tracker-rescue:R-Device
- gave numbers to parts that had none: 6
Connections:
- net Earth: now also R7.1
- net LED: now reaches U4.11 (IO26)
- net LED: now also D3.2 (A)
- new net: D3.1 (K), R7.2
Changed lines of the file:
@@
 BOOT
 $Comp
-L Device:Q_NPN_BEC Q?
+L Device:Q_NPN_BEC Q1
 U 1 1 6114B2B0
 P 8500 3800
-F 0 "Q?" H 8690 3846 50  0000 L CNN
+F 0 "Q1" H 8690 3846 50  0000 L CNN
 F 1 "S8050" H 8690 3755 50  0000 L CNN
 F 2 "Package_TO_SOT_SMD:SOT-23" H 8700 3900 50  0001 C CNN
@@
 $EndComp
 $Comp
-L cat_tracker-rescue:R-Device R?
+L cat_tracker-rescue:R-Device R6
 U 1 1 6114D548
 P 8150 3800
-F 0 "R?" V 8050 3750 50  0000 L CNN
+F 0 "R6" V 8050 3750 50  0000 L CNN
 F 1 "100" V 8150 3800 50  0000 C CNN
 F 2 "Resistor_SMD:R_0603_1608Metric_Pad0.98x0.95mm_HandSolder" V 8080 3800 50  0001 C CNN
@@
 $EndComp
 $Comp
-L cat_tracker-rescue:Earth-power #PWR?
+L cat_tracker-rescue:Earth-power #PWR02
 U 1 1 61152057
 P 8600 4000
-F 0 "#PWR?" H 8600 3750 50  0001 C CNN
+F 0 "#PWR02" H 8600 3750 50  0001 C CNN
 F 1 "Earth" H 8600 3850 50  0001 C CNN
 F 2 "" H 8600 4000 50  0001 C CNN
@@
 $EndComp
 $Comp
-L Connector_Generic:Conn_01x03 J?
+L Connector_Generic:Conn_01x03 J3
 U 1 1 61153F36
 P 9200 3300
-F 0 "J?" H 9280 3342 50  0000 L CNN
+F 0 "J3" H 9280 3342 50  0000 L CNN
 F 1 "GP2Y0A41SK0F" H 9280 3251 50  0000 L CNN
 F 2 "Connector_JST:JST_PH_S3B-PH-K_1x03_P2.00mm_Horizontal" H 9200 3300 50  0001 C CNN
@@
 IR_EN
 $Comp
-L cat_tracker-rescue:SW_Push-Switch SW?
+L cat_tracker-rescue:SW_Push-Switch SW3
 U 1 1 6115D292
 P 8650 5100
-F 0 "SW?" H 8650 5385 50  0000 C CNN
+F 0 "SW3" H 8650 5385 50  0000 C CNN
 F 1 "Pairing Btn" H 8650 5294 50  0000 C CNN
 F 2 "ali_Switch:NW3-A03-05" H 8650 5300 50  0001 C CNN
@@
 $EndComp
 $Comp
-L cat_tracker-rescue:+3.3V-power #PWR?
+L cat_tracker-rescue:+3.3V-power #PWR01
 U 1 1 6115D298
 P 8350 5000
-F 0 "#PWR?" H 8350 4850 50  0001 C CNN
+F 0 "#PWR01" H 8350 4850 50  0001 C CNN
 F 1 "+3.3V" H 8365 5173 50  0000 C CNN
 F 2 "" H 8350 5000 50  0001 C CNN
@@
 	8350 5100 8450 5100
 $Comp
-L cat_tracker-rescue:C-Device C?
+L cat_tracker-rescue:C-Device C8
 U 1 1 6115D2A0
 P 8850 5250
-F 0 "C?" H 8965 5296 50  0000 L CNN
+F 0 "C8" H 8965 5296 50  0000 L CNN
 F 1 "100n" H 8965 5205 50  0000 L CNN
 F 2 "Capacitor_SMD:C_0603_1608Metric_Pad1.08x0.95mm_HandSolder" H 8888 5100 50  0001 C CNN
@@
 $EndComp
 $Comp
-L cat_tracker-rescue:R-Device R?
+L cat_tracker-rescue:R-Device R8
 U 1 1 6115D2A6
 P 9000 5100
-F 0 "R?" V 8900 5050 50  0000 L CNN
+F 0 "R8" V 8900 5050 50  0000 L CNN
 F 1 "1k" V 9000 5100 50  0000 C CNN
 F 2 "Resistor_SMD:R_0603_1608Metric_Pad0.98x0.95mm_HandSolder" V 8930 5100 50  0001 C CNN
@@
 Connection ~ 8850 5100
 $Comp
-L cat_tracker-rescue:Earth-power #PWR?
+L cat_tracker-rescue:Earth-power #PWR03
 U 1 1 6115D2AD
 P 8850 5400
-F 0 "#PWR?" H 8850 5150 50  0001 C CNN
+F 0 "#PWR03" H 8850 5150 50  0001 C CNN
 F 1 "Earth" H 8850 5250 50  0001 C CNN
 F 2 "" H 8850 5400 50  0001 C CNN
@@
 Text GLabel 6150 5200 2    50   Input ~ 0
 BTN
+Text GLabel 6150 5100 2    50   Input ~ 0
+LED
+$Comp
+L Device:LED D3
+U 1 1 6115FD9F
+P 8450 5950
+F 0 "D3" H 8443 5695 50  0000 C CNN
+F 1 "LED" H 8443 5786 50  0000 C CNN
+F 2 "LED_SMD:LED_0805_2012Metric_Pad1.15x1.40mm_HandSolder" H 8450 5950 50  0001 C CNN
+F 3 "~" H 8450 5950 50  0001 C CNN
+	1    8450 5950
+	-1   0    0    1
+$EndComp
+$Comp
+L cat_tracker-rescue:R-Device R7
+U 1 1 611600BC
+P 8750 5950
+F 0 "R7" V 8650 5900 50  0000 L CNN
+F 1 "1k" V 8750 5950 50  0000 C CNN
+F 2 "Resistor_SMD:R_0603_1608Metric_Pad0.98x0.95mm_HandSolder" V 8680 5950 50  0001 C CNN
+F 3 "~" H 8750 5950 50  0001 C CNN
+	1    8750 5950
+	0    1    1    0
+$EndComp
+$Comp
+L cat_tracker-rescue:Earth-power #PWR04
+U 1 1 61160B6E
+P 8900 5950
+F 0 "#PWR04" H 8900 5700 50  0001 C CNN
+F 1 "Earth" H 8900 5800 50  0001 C CNN
+F 2 "" H 8900 5950 50  0001 C CNN
+F 3 "~" H 8900 5950 50  0001 C CNN
+	1    8900 5950
+	0    -1   -1   0
+$EndComp
+Text GLabel 8300 5950 0    50   Input ~ 0
+LED
 $EndSCHEMATC

Commit message: 2021-08-29
Parts:
- C1: symbol cat_tracker-rescue:C-Device -> cat_toilet-rescue:C-Device-cat_tracker-rescue; MPN (none) -> TPCL106K010R4000
- C2, C3, C4, C5, C6, C7, C8: symbol cat_tracker-rescue:C-Device -> cat_toilet-rescue:C-Device-cat_tracker-rescue
- D1: value SK24/SMA -> SK24/SMB; footprint Diode_SMD:D_SMA_Handsoldering -> Diode_SMD:D_SMB_Handsoldering; symbol cat_tracker-rescue:D_Schottky-Device -> cat_toilet-rescue:D_Schottky-Device-cat_tracker-rescue; MPN (none) -> SK24-TP
- D2: symbol cat_tracker-rescue:LED-Device -> cat_toilet-rescue:LED-Device-cat_tracker-rescue
- J1: symbol cat_tracker-rescue:Conn_01x02-Connector_Generic -> cat_toilet-rescue:Conn_01x02-Connector_Generic-cat_tracker-rescue
- J2: symbol cat_tracker-rescue:Conn_01x04-Connector_Generic -> cat_toilet-rescue:Conn_01x04-Connector_Generic-cat_tracker-rescue
- R1, R2, R3, R4, R5, R6, R7, R8: symbol cat_tracker-rescue:R-Device -> cat_toilet-rescue:R-Device-cat_tracker-rescue
- SW1, SW2, SW3: symbol cat_tracker-rescue:SW_Push-Switch -> cat_toilet-rescue:SW_Push-Switch-cat_tracker-rescue
- U2: MPN (none) -> CType Connector
- U3: symbol cat_tracker-rescue:MCP73831-2-OT-Battery_Management -> cat_toilet-rescue:MCP73831-2-OT-Battery_Management-cat_tracker-rescue
- U4: symbol cat_tracker-rescue:ESP32-WROOM-32D-RF_Module -> cat_toilet-rescue:ESP32-WROOM-32D-RF_Module-cat_tracker-rescue
Changed lines of the file:
@@
 $EndDescr
 $Comp
-L cat_tracker-rescue:ESP32-WROOM-32D-RF_Module U4
+L cat_toilet-rescue:ESP32-WROOM-32D-RF_Module-cat_tracker-rescue U4
 U 1 1 61108DF0
 P 5550 4500
@@
 F 2 "ali_Connector:USB_CType_6Pin" H 2050 1500 50  0001 C CNN
 F 3 "" H 2050 1500 50  0001 C CNN
+F 4 "CType Connector" H 2050 1500 50  0001 C CNN "MPN"
 	1    2050 1500
 	1    0    0    -1
 $EndComp
 $Comp
-L cat_tracker-rescue:MCP73831-2-OT-Battery_Management U3
+L cat_toilet-rescue:MCP73831-2-OT-Battery_Management-cat_tracker-rescue U3
 U 1 1 6110E339
 P 4800 1500
@@
 $EndComp
 $Comp
-L cat_tracker-rescue:D_Schottky-Device D1
+L cat_toilet-rescue:D_Schottky-Device-cat_tracker-rescue D1
 U 1 1 611100B7
 P 4550 1000
 F 0 "D1" H 4550 783 50  0000 C CNN
-F 1 "SK24/SMA" H 4550 874 50  0000 C CNN
-F 2 "Diode_SMD:D_SMA_Handsoldering" H 4550 1000 50  0001 C CNN
-F 3 "~" H 4550 1000 50  0001 C CNN
+F 1 "SK24/SMB" H 4550 874 50  0000 C CNN
+F 2 "Diode_SMD:D_SMB_Handsoldering" H 4550 1000 50  0001 C CNN
+F 3 "https://www.mouser.com/ProductDetail/Micro-Commercial-Components-MCC/SK24-TP?qs=ekjJs1tcck0x%252BNZEMIWSMw%3D%3D" H 4550 1000 50  0001 C CNN
+F 4 "SK24-TP" H 4550 1000 50  0001 C CNN "MPN"
 	1    4550 1000
 	-1   0    0    1
 $EndComp
 $Comp
-L cat_tracker-rescue:C-Device C1
+L cat_toilet-rescue:C-Device-cat_tracker-rescue C1
 U 1 1 6111090E
 P 2700 1500
@@
 F 1 "10u" H 2815 1455 50  0000 L CNN
 F 2 "Capacitor_SMD:C_0603_1608Metric_Pad1.08x0.95mm_HandSolder" H 2738 1350 50  0001 C CNN
-F 3 "~" H 2700 1500 50  0001 C CNN
+F 3 "https://www.mouser.com/ProductDetail/AVX/TPCL106K010R4000?qs=sGAEpiMZZMukHu%252BjC5l7YbWrvsR5dLklJIeP7A7npOo%3D" H 2700 1500 50  0001 C CNN
+F 4 "TPCL106K010R4000" H 2700 1500 50  0001 C CNN "MPN"
 	1    2700 1500
 	1    0    0    -1
 $EndComp
 $Comp
-L cat_tracker-rescue:C-Device C2
+L cat_toilet-rescue:C-Device-cat_tracker-rescue C2
 U 1 1 61112178
 P 3150 1500
@@
 	2350 1650 2250 1650
 $Comp
-L cat_tracker-rescue:Earth-power #PWR0101
+L cat_toilet-rescue:Earth-power-cat_tracker-rescue #PWR0101
 U 1 1 61112600
 P 2250 1750
@@
 $EndComp
 $Comp
-L cat_tracker-rescue:Earth-power #PWR0102
+L cat_toilet-rescue:Earth-power-cat_tracker-rescue #PWR0102
 U 1 1 6111274F
 P 2250 1250
@@
 $EndComp
 $Comp
-L cat_tracker-rescue:Earth-power #PWR0103
+L cat_toilet-rescue:Earth-power-cat_tracker-rescue #PWR0103
 U 1 1 61112BC4
 P 2700 1650
@@
 $EndComp
 $Comp
-L cat_tracker-rescue:Earth-power #PWR0104
+L cat_toilet-rescue:Earth-power-cat_tracker-rescue #PWR0104
 U 1 1 611130BC
 P 3150 1650
@@
 VBUS
 $Comp
-L cat_tracker-rescue:LED-Device D2
+L cat_toilet-rescue:LED-Device-cat_tracker-rescue D2
 U 1 1 61114FC1
 P 5050 1000
@@
 $EndComp
 $Comp
-L cat_tracker-rescue:R-Device R1
+L cat_toilet-rescue:R-Device-cat_tracker-rescue R1
 U 1 1 61115A90
 P 5400 1150
@@
 $EndComp
 $Comp
-L cat_tracker-rescue:R-Device R3
+L cat_toilet-rescue:R-Device-cat_tracker-rescue R3
 U 1 1 6111654E
 P 4300 1750
@@
 $EndComp
 $Comp
-L cat_tracker-rescue:C-Device C5
+L cat_toilet-rescue:C-Device-cat_tracker-rescue C5
 U 1 1 61116BD2
 P 5650 1550
@@
 $EndComp
 $Comp
-L cat_tracker-rescue:Earth-power #PWR0105
+L cat_toilet-rescue:Earth-power-cat_tracker-rescue #PWR0105
 U 1 1 611173E7
 P 4300 1900
@@
 $EndComp
 $Comp
-L cat_tracker-rescue:Earth-power #PWR0106
+L cat_toilet-rescue:Earth-power-cat_tracker-rescue #PWR0106
 U 1 1 6111791D
 P 4800 1800
@@
 	5200 1400 5650 1400
 $Comp
-L cat_tracker-rescue:Earth-power #PWR0107
+L cat_toilet-rescue:Earth-power-cat_tracker-rescue #PWR0107
 U 1 1 61118BDB
 P 5650 1700
@@
 	4300 1600 4400 1600
 $Comp
-L cat_tracker-rescue:Conn_01x02-Connector_Generic J1
+L cat_toilet-rescue:Conn_01x02-Connector_Generic-cat_tracker-rescue J1
 U 1 1 6111965B
 P 6300 1400
@@
 $EndComp
 $Comp
-L cat_tracker-rescue:Earth-power #PWR0108
+L cat_toilet-rescue:Earth-power-cat_tracker-rescue #PWR0108
 U 1 1 61119EBD
 P 6000 1600
@@
 $EndComp
 $Comp
-L cat_tracker-rescue:C-Device C3
+L cat_toilet-rescue:C-Device-cat_tracker-rescue C3
 U 1 1 6111DBE3
 P 7300 1500
@@
 	7650 1350 7750 1350
 $Comp
-L cat_tracker-rescue:Earth-power #PWR0109
+L cat_toilet-rescue:Earth-power-cat_tracker-rescue #PWR0109
 U 1 1 6111EF7B
 P 7300 1650
@@
 $EndComp
 $Comp
-L cat_tracker-rescue:Earth-power #PWR0110
+L cat_toilet-rescue:Earth-power-cat_tracker-rescue #PWR0110
 U 1 1 6111F802
 P 7650 1650
@@
 	7650 1550 7750 1550
 $Comp
-L cat_tracker-rescue:R-Device R2
+L cat_toilet-rescue:R-Device-cat_tracker-rescue R2
 U 1 1 61120B43
 P 8650 1500
@@
 	8450 1550 8350 1550
 $Comp
-L cat_tracker-rescue:+3.3V-power #PWR0111
+L cat_toilet-rescue:+3.3V-power-cat_tracker-rescue #PWR0111
 U 1 1 611226CB
 P 8950 1350
@@
 $EndComp
 $Comp
-L cat_tracker-rescue:C-Device C4
+L cat_toilet-rescue:C-Device-cat_tracker-rescue C4
 U 1 1 61123213
 P 8950 1500
@@
 Connection ~ 8650 1350
 $Comp
-L cat_tracker-rescue:Earth-power #PWR0112
+L cat_toilet-rescue:Earth-power-cat_tracker-rescue #PWR0112
 U 1 1 611243DC
 P 8950 1650
@@
 $EndComp
 $Comp
-L cat_tracker-rescue:+3.3V-power #PWR0113
+L cat_toilet-rescue:+3.3V-power-cat_tracker-rescue #PWR0113
 U 1 1 61124907
 P 5550 3100
@@
 EN
 $Comp
-L cat_tracker-rescue:Earth-power #PWR0114
+L cat_toilet-rescue:Earth-power-cat_tracker-rescue #PWR0114
 U 1 1 61126409
 P 5550 5900
@@
 NoConn ~ 6150 3700
 $Comp
-L cat_tracker-rescue:SW_Push-Switch SW1
+L cat_toilet-rescue:SW_Push-Switch-cat_tracker-rescue SW1
 U 1 1 6115F88F
 P 1600 3300
@@
 $EndComp
 $Comp
-L cat_tracker-rescue:+3.3V-power #PWR0128
+L cat_toilet-rescue:+3.3V-power-cat_tracker-rescue #PWR0128
 U 1 1 6115FA35
 P 1300 3200
@@
 	1300 3300 1400 3300
 $Comp
-L cat_tracker-rescue:Conn_01x04-Connector_Generic J2
+L cat_toilet-rescue:Conn_01x04-Connector_Generic-cat_tracker-rescue J2
 U 1 1 611619C1
 P 1600 4450
@@
 $EndComp
 $Comp
-L cat_tracker-rescue:+3.3V-power #PWR0129
+L cat_toilet-rescue:+3.3V-power-cat_tracker-rescue #PWR0129
 U 1 1 61162905
 P 1800 4350
@@
 $EndComp
 $Comp
-L cat_tracker-rescue:Earth-power #PWR0130
+L cat_toilet-rescue:Earth-power-cat_tracker-rescue #PWR0130
 U 1 1 611632DD
 P 1800 4450
@@
 TX
 $Comp
-L cat_tracker-rescue:C-Device C6
+L cat_toilet-rescue:C-Device-cat_tracker-rescue C6
 U 1 1 6116473C
 P 1800 3450
@@
 $EndComp
 $Comp
-L cat_tracker-rescue:R-Device R4
+L cat_toilet-rescue:R-Device-cat_tracker-rescue R4
 U 1 1 61164D5E
 P 1950 3300
@@
 Connection ~ 1800 3300
 $Comp
-L cat_tracker-rescue:Earth-power #PWR0131
+L cat_toilet-rescue:Earth-power-cat_tracker-rescue #PWR0131
 U 1 1 611655D5
 P 1800 3600
@@
 BOOT
 $Comp
-L cat_tracker-rescue:SW_Push-Switch SW2
+L cat_toilet-rescue:SW_Push-Switch-cat_tracker-rescue SW2
 U 1 1 6116806C
 P 2800 3300
@@
 $EndComp
 $Comp
-L cat_tracker-rescue:+3.3V-power #PWR0132
+L cat_toilet-rescue:+3.3V-power-cat_tracker-rescue #PWR0132
 U 1 1 61168072
 P 2500 3200
@@
 	2500 3300 2600 3300
 $Comp
-L cat_tracker-rescue:C-Device C7
+L cat_toilet-rescue:C-Device-cat_tracker-rescue C7
 U 1 1 6116807A
 P 3000 3450
@@
 $EndComp
 $Comp
-L cat_tracker-rescue:R-Device R5
+L cat_toilet-rescue:R-Device-cat_tracker-rescue R5
 U 1 1 61168080
 P 3150 3300
@@
 Connection ~ 3000 3300
 $Comp
-L cat_tracker-rescue:Earth-power #PWR0133
+L cat_toilet-rescue:Earth-power-cat_tracker-rescue #PWR0133
 U 1 1 61168087
 P 3000 3600
@@
 $EndComp
 $Comp
-L cat_tracker-rescue:R-Device R6
+L cat_toilet-rescue:R-Device-cat_tracker-rescue R6
 U 1 1 6114D548
 P 8150 3800
@@
 $EndComp
 $Comp
-L cat_tracker-rescue:Earth-power #PWR02
+L cat_toilet-rescue:Earth-power-cat_tracker-rescue #PWR02
 U 1 1 61152057
 P 8600 4000
@@
 IR_EN
 $Comp
-L cat_tracker-rescue:SW_Push-Switch SW3
+L cat_toilet-rescue:SW_Push-Switch-cat_tracker-rescue SW3
 U 1 1 6115D292
 P 8650 5100
@@
 $EndComp
 $Comp
-L cat_tracker-rescue:+3.3V-power #PWR01
+L cat_toilet-rescue:+3.3V-power-cat_tracker-rescue #PWR01
 U 1 1 6115D298
 P 8350 5000
@@
 	8350 5100 8450 5100
 $Comp
-L cat_tracker-rescue:C-Device C8
+L cat_toilet-rescue:C-Device-cat_tracker-rescue C8
 U 1 1 6115D2A0
 P 8850 5250
@@
 $EndComp
 $Comp
-L cat_tracker-rescue:R-Device R8
+L cat_toilet-rescue:R-Device-cat_tracker-rescue R8
 U 1 1 6115D2A6
 P 9000 5100
@@
 Connection ~ 8850 5100
 $Comp
-L cat_tracker-rescue:Earth-power #PWR03
+L cat_toilet-rescue:Earth-power-cat_tracker-rescue #PWR03
 U 1 1 6115D2AD
 P 8850 5400
@@
 $EndComp
 $Comp
-L cat_tracker-rescue:R-Device R7
+L cat_toilet-rescue:R-Device-cat_tracker-rescue R7
 U 1 1 611600BC
 P 8750 5950
@@
 $EndComp
 $Comp
-L cat_tracker-rescue:Earth-power #PWR04
+L cat_toilet-rescue:Earth-power-cat_tracker-rescue #PWR04
 U 1 1 61160B6E
 P 8900 5950

Commit message: 2021-12-14
Parts:
- removed C4: 10u, Capacitor_SMD:C_0603_1608Metric_Pad1.08x0.95mm_HandSolder, symbol cat_toilet-rescue:C-Device-cat_tracker-rescue
- removed D1: SK24/SMB, Diode_SMD:D_SMB_Handsoldering, symbol cat_toilet-rescue:D_Schottky-Device-cat_tracker-rescue
- removed D2: LED/2012, LED_SMD:LED_0805_2012Metric_Pad1.15x1.40mm_HandSolder, symbol cat_toilet-rescue:LED-Device-cat_tracker-rescue
- removed SW3: Pairing Btn, ali_Switch:NW3-A03-05, symbol cat_toilet-rescue:SW_Push-Switch-cat_tracker-rescue
- removed U1: NCP187, Package_DFN_QFN:DFN-6-1EP_2x2mm_P0.65mm_EP1x1.6mm, symbol add_LDO:NCP187
- removed U2: USB_CType_6Pin, ali_Connector:USB_CType_6Pin, symbol ali_Connector:USB_CType_6Pin
- added C9: 1u, Capacitor_SMD:C_0603_1608Metric, symbol cat_toilet-rescue:C-Device-cat_tracker-rescue
- added D1: LED/1608, LED_SMD:LED_0603_1608Metric, symbol Device:LED
- added Q2, Q3: BC856B,215, Package_TO_SOT_SMD:SOT-23, symbol Device:Q_PNP_BEC
- added R10, R11, R9: 33k, Resistor_SMD:R_0603_1608Metric, symbol cat_toilet-rescue:R-Device-cat_tracker-rescue
- added TP1: TestPoint_2Pole, tp:boot, symbol Connector:TestPoint_2Pole
- added U1: MCP100-315D, Package_TO_SOT_SMD:SOT-23, symbol Power_Supervisor:MCP100-315D
- added U2: USB_CType_2Pin, ali_Connector:USB_CType_2Pin, symbol ali_Connector:USB_CType_2Pin
- added U5: MCP1802T-3302I/OT, Package_TO_SOT_SMD:SOT-23-5, symbol MIC531833YD5TR:MIC5318-3.3YD5-TR
- C1: footprint Capacitor_SMD:C_0603_1608Metric_Pad1.08x0.95mm_HandSolder -> Capacitor_SMD:C_0603_1608Metric; MPN TPCL106K010R4000 -> 302010103
- C2, C3, C6, C7, C8: footprint Capacitor_SMD:C_0603_1608Metric_Pad1.08x0.95mm_HandSolder -> Capacitor_SMD:C_0603_1608Metric; MPN (none) -> 302010138
- C5: footprint Capacitor_SMD:C_0603_1608Metric_Pad1.08x0.95mm_HandSolder -> Capacitor_SMD:C_0603_1608Metric; MPN (none) -> 302010103
- D3: value LED -> LED/1608; footprint LED_SMD:LED_0805_2012Metric_Pad1.15x1.40mm_HandSolder -> LED_SMD:LED_0603_1608Metric; MPN (none) -> SMLEN3WBC8W1
- J1: value Conn_01x02 -> Batt; footprint Connector_Molex:Molex_PicoBlade_53261-0271_1x02-1MP_P1.25mm_Horizontal -> tp:boot
- J2: footprint Connector_PinHeader_2.54mm:PinHeader_1x04_P2.54mm_Vertical -> Connector_PinHeader_2.00mm:PinHeader_1x04_P2.00mm_Vertical
- J3: footprint Connector_JST:JST_PH_S3B-PH-K_1x03_P2.00mm_Horizontal -> Connector_JST:JST_PH_B3B-PH-K_1x03_P2.00mm_Vertical
- Q1: value S8050 -> npn; MPN (none) -> BC846A,215
- R1: value 510 -> 10k; footprint Resistor_SMD:R_0603_1608Metric_Pad0.98x0.95mm_HandSolder -> Resistor_SMD:R_0603_1608Metric; MPN (none) -> 301010293
- R2: value 100k -> 33k; footprint Resistor_SMD:R_0603_1608Metric_Pad0.98x0.95mm_HandSolder -> Resistor_SMD:R_0603_1608Metric; MPN (none) -> CR0603JA0333G
- R3: footprint Resistor_SMD:R_0603_1608Metric_Pad0.98x0.95mm_HandSolder -> Resistor_SMD:R_0603_1608Metric; MPN (none) -> 301010113
- R4: value 1k -> 0; footprint Resistor_SMD:R_0603_1608Metric_Pad0.98x0.95mm_HandSolder -> Resistor_SMD:R_0603_1608Metric; MPN (none) -> 301011968
- R5: value 1k -> 10k; MPN (none) -> 301010293
- R6: footprint Resistor_SMD:R_0603_1608Metric_Pad0.98x0.95mm_HandSolder -> Resistor_SMD:R_0603_1608Metric; MPN (none) -> 301011976
- R7, R8: footprint Resistor_SMD:R_0603_1608Metric_Pad0.98x0.95mm_HandSolder -> Resistor_SMD:R_0603_1608Metric; MPN (none) -> 301010291
- SW1: footprint ali_Switch:NW3-A03-05 -> Button_Switch_SMD:SW_SPST_B3U-1000P
- SW2: value EN Btn -> Pairing Btn; footprint ali_Switch:NW3-A03-05 -> Button_Switch_SMD:SW_SPST_B3U-1000P; MPN (none) -> B3U-1000P
- U3: MPN (none) -> MCP73831T-2ACI/OT
- U4: MPN ESP32-WROOM-32E -> ESP32-WROOM-32E(M113EH3200PH3Q0)
Connections:
- net +3V3: now also C7.1, R1.2, R5.2, Q2.2 (E), Q3.2 (E), R10.2, R11.2, U5.5 (OUT); no longer R2.1, SW1.1
- net BATT: now also U1.2 (VDD), U5.1 (IN)
- net BOOT: now also TP1.2
- net EN: now also R1.1, C9.1
- net Earth: now also SW1.1, C9.2, TP1.1, U1.3 (VSS), U2.12 (GND), U5.2 (GND)
- net LED: now also R9.1; no longer D3.2 (A)
- net VBUS: now also U3.4 (VDD), U2.9 (VBUS)
- net CHRG: now reaches U3.1 (STAT)
- net CHRG: now also R2.1; no longer R1.2
- net at R2.2: now also Q2.1 (B), R10.1
- net at C8.1, R8.2: now also SW2.2
- net at D3.1 (K), R7.2: now also D1.1 (K)
- new net: D1.2 (A), D3.2 (A), Q2.3 (C), Q3.3 (C)
- new net: U1.1 (~RST), U5.3 (EN)
- new net: Q3.1 (B), R11.1, R9.2
- no-connect marks 4 -> 5
Other:
- moved on the sheet: C3, C6, C8, D3, J2, R4, R5, R7, R8, SW1
